File: Designs/PCB/KiCad/Projects/Test_1.sch (KiCad schematic (older format))
At the start: 4 parts

Commit message: Importing EasyEda Desgns in KiCad
Parts:
- added U?: STM32, symbol STM32
- added U?: LoRa, symbol LoRa
Changed lines of the file:
@@
+	1    0    0    -1
+$EndComp
+$Comp
+L STM32 U?
+U 1 1 5F084833
+P 3300 4650
+F 0 "U?" H 4100 5350 60  0000 C CNN
+F 1 "STM32" H 3300 4550 118 0000 C CNN
+F 2 "" H 3300 4650 60  0001 C CNN
+F 3 "" H 3300 4650 60  0001 C CNN
+	1    3300 4650
+	1    0    0    -1
+$EndComp
+$Comp
+L LoRa U?
+U 1 1 5F08489C
+P 5750 5000
+F 0 "U?" H 5750 4550 60  0000 C CNN
+F 1 "LoRa" H 5750 5100 60  0000 C CNN
+F 2 "" H 5750 4550 60  0001 C CNN
+F 3 "" H 5750 4550 60  0001 C CNN
+	1    5750 5000
 	1    0    0    -1
 $EndComp
