File: Designs/PCB/KiCad/Projects/Test_1/Test_2/Blue Pill/BluePill_module/BluePill_module.sch (KiCad schematic (older format))
At the start: 13 parts, among them Y1 32.768K, Y2 8Mhz

Commit message: Update
Changed lines of the file:
@@
 	3850 4750 3450 4750
-$Comp
-L power:GNDREF #PWR?
-U 1 1 5F0FB70B
-P 2750 4750
-F 0 "#PWR?" H 2755 4577 50  0001 C CNN
-F 1 "GNDREF" H 2755 4577 50  0000 C CNN
-F 2 "" H 2750 4750 50  0001 C CNN
-F 3 "" H 2750 4750 50  0001 C CNN
-	1    2750 4750
-	1    0    0    -1
-$EndComp
-Wire Wire Line
-	3150 4750 2750 4750
-Connection ~ 3150 4750
 $Comp
 L Connector_Generic:Conn_02x03_Top_Bottom J?
@@
 Wire Wire Line
 	1950 3750 2250 3750
+Text Label 1850 4150 0    50   ~ 0
+GND
+Wire Wire Line
+	1650 4150 1850 4150
+Connection ~ 1650 4150
+Text Label 2800 4750 0    50   ~ 0
+GND
+Wire Wire Line
+	2800 4750 3150 4750
+Connection ~ 3150 4750
 $EndSCHEMATC

Commit message: Update
Parts:
- added J?: Prog Hdr, symbol Connector_Generic:Conn_01x05
Connections:
- net +5V: now also J?.4 (Pin_4)
- net GNDREF: now also J?.5 (Pin_5)
- net VCC3V3: now also J?.3 (Pin_3)
- net TX0: now reaches U?.30 (PA9)
- net TX0: now also J?.1 (Pin_1)
- net RX0: now reaches U?.31 (PA10)
- net RX0: now also J?.2 (Pin_2)
Changed lines of the file:
@@
 U 1 1 5F0D833D
 P 6400 3350
-F 0 "U?" H 7594 3246 60  0000 L CNN
-F 1 "STM32" H 7594 3097 118 0000 L CNN
+F 0 "U?" H 7400 4250 60  0000 L CNN
+F 1 "STM32" H 6250 3050 118 0000 L CNN
 F 2 "" H 6400 3350 60  0001 C CNN
 F 3 "" H 6400 3350 60  0001 C CNN
@@
 	2800 4750 3150 4750
 Connection ~ 3150 4750
+$Comp
+L Connector_Generic:Conn_01x05 J?
+U 1 1 5F0DE12E
+P 8150 1750
+F 0 "J?" H 8068 1325 50  0000 C CNN
+F 1 "Prog Hdr" H 8068 1416 50  0000 C CNN
+F 2 "" H 8150 1750 50  0001 C CNN
+F 3 "~" H 8150 1750 50  0001 C CNN
+	1    8150 1750
+	-1   0    0    1
+$EndComp
+Text Label 8550 1550 2    50   ~ 0
+GND
+Text Label 950  3750 0    50   ~ 0
+5V
+Wire Wire Line
+	950  3750 1150 3750
+Connection ~ 1150 3750
+Text Label 8650 1650 2    50   ~ 0
+5V
+Text Label 8850 1750 2    50   ~ 0
+VCC3V3
+Wire Wire Line
+	8350 1550 8550 1550
+Wire Wire Line
+	8650 1650 8350 1650
+Wire Wire Line
+	8350 1750 8850 1750
+Text Label 7900 3600 2    50   ~ 0
+TX0
+Wire Wire Line
+	7550 3600 7900 3600
+Text Label 7900 3500 2    50   ~ 0
+RX0
+Wire Wire Line
+	7900 3500 7550 3500
+Text Label 8700 1850 2    50   ~ 0
+RX0
+Text Label 8700 1950 2    50   ~ 0
+TX0
+Wire Wire Line
+	8700 1950 8350 1950
+Wire Wire Line
+	8350 1850 8700 1850
 $EndSCHEMATC
