File: Designs/PCB/KiCad/Projects/SwitchBoard/FrontEnd_4S/FrontEnd_4S.sch (KiCad schematic (older format))
At the start: 21 parts, among them J1 Header 3x2, J2 Prog Hdr, SW1 SW_Push, U1 APK2112.K-3.3, U2 STM32, Y1 32.768K, Y2 8Mhz

Commit message: update
Parts:
- removed R2: 1M, Resistors_SMD:R_0805, symbol Device:R
- removed U2: STM32, Custom_Libraries:STM32(LQFP48), symbol stm32:STM32
- added C10, C11, C8, C9: 100 nf, Capacitors_SMD:C_0805, symbol Device:C
- added C12, C13, C14, C15: 10uf, Capacitors_SMD:C_0805, symbol Device:C
- added J3: Header_In, Pin_Headers:Pin_Header_Straight_1x08_Pitch2.54mm, symbol Connector:Conn_01x08_Female
- added J?: Conn_01x05_Female, symbol Connector:Conn_01x05_Female
- added T1, T2, T3, T4: Touch_Pad, Custom_Libraries:Touch_Pad, symbol touch_pad:Touch_Pad
- added U4, U5, U6, U7: TTP223, TO_SOT_Packages_SMD:SOT-23-6, symbol Switch:TTP223
- added U?: STM32, Custom_Libraries:STM32WB55CEU6, symbol STM32WB55CEU6:STM32WB55CEU6
- C2, C3: value 20pf -> 10pf
- D1: renamed from D?; footprint (none) -> Diodes_SMD:D_0805
- J1: symbol Connector_Generic:Conn_02x03_Top_Bottom -> Connector_Generic:Conn_02x03_Counter_Clockwise
- U3: renamed from U?; footprint (none) -> Custom_Libraries:LoRa
- Y2: value 8Mhz -> 32Mhz
- gave numbers to parts that had none: 5
Connections:
- net labels added: DSW_1, DSW_2, DSW_3, DSW_4, Energy, Opto_IN, Reset_Lora, Touch_1, Touch_2, Touch_3, Touch_4
- net labels removed: GNDREF, Reset
- wire segments 108 -> 187
- no-connect marks 4 -> 12
Other:
- note added: "Input / Output Headers"
- note added: "Touch Pads"
- moved on the sheet: AE1, C2, C3, C4, C5, J2, J4, U3, Y1, Y2
