File: Designs/PCB/KiCad/Projects/SwitchBoard/FrontEnd_4S/_autosave-FrontEnd_4S.sch (KiCad schematic (older format))
At the start: 38 parts, among them J1 Header 3x2, J2 Prog Hdr, J3 Header_In, J4 SWD, SW1 SW_Push, T1 Touch_Pad, T2 Touch_Pad, T3 Touch_Pad, T4 Touch_Pad, U1 APK2112.K-3.3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

Commit message: update
Parts:
- removed J4: SWD, Pin_Headers:Pin_Header_Straight_1x04_Pitch2.54mm, symbol Connector:Conn_01x04_Female
- removed R2: 1M, Resistors_SMD:R_0805, symbol Device:R
- removed U2: STM32, Custom_Libraries:STM32(LQFP48), symbol stm32:STM32
- added J?: Conn_01x05_Female, symbol Connector:Conn_01x05_Female
- added U?: STM32, Custom_Libraries:STM32WB55CEU6, symbol STM32WB55CEU6:STM32WB55CEU6
- C2, C3: value 20pf -> 10pf
- J1: symbol Connector_Generic:Conn_02x03_Top_Bottom -> Connector_Generic:Conn_02x03_Counter_Clockwise
- Y2: value 8Mhz -> 32Mhz
Connections:
- net labels added: Reset_Lora
- net labels removed: GNDREF, Reset
- wire segments 170 -> 183
- no-connect marks 16 -> 12
Other:
- note added: "ST-Link conn"
