File: Designs/PCB/KiCad/Projects/SwitchBoard/Sensor_pcb/Sensor_all/Sensor_pcb_v1/Sensor_pcb_v1.kicad_pcb (KiCad board)
At the start: 2 copper layers, 29 parts, among them J1 Header 3x2, J2 Prog Hdr, J3 Solar_input, J4 SWD, J5 Battery_input, SW1 SW_Push, SW2 SW_Push, U1 APK2112.K-3.3, U2 STM32, U3 LoRa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

Commit message: update
Parts:
- moved R4 89.3 mm to (52.0, 21.1)
- moved AE1 89.3 mm to (66.0, 58.6)
- moved J2 89.3 mm to (66.0, 32.6)
- moved J3 89.3 mm to (25.6, 57.1)
- moved SW2 89.3 mm to (35.0, 56.1)
- moved C1 89.3 mm to (36.5, 32.6)
- moved C2 89.3 mm to (39.0, 26.6)
- moved C3 89.3 mm to (45.5, 30.6)
- moved C4 89.3 mm to (48.0, 30.6)
- moved C5 89.3 mm to (39.0, 29.1)
- moved C6 89.3 mm to (32.0, 60.6)
- moved C7 89.3 mm to (31.0, 43.1)
- moved D1 89.3 mm to (37.0, 51.6)
- moved D2 89.3 mm to (32.0, 57.1)
- moved J1 89.3 mm to (61.5, 25.1)
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
Commit message: Update
Parts:
- added J6: Distance /, Pin_Headers:Pin_Header_Straight_1x04_Pitch2.54mm, F.Cu at (60.2, 34.0)
- added R6: 2.7K, Resistors_SMD:R_0805, B.Cu at (55.8, 36.8)
- added R7: 4.7K, Resistors_SMD:R_0805, B.Cu at (55.0, 41.7)
- AE1: value Antenna -> ANT; footprint SMD_Packages:1Pin -> Pin_Headers:Pin_Header_Straight_1x01_Pitch2.54mm
- D1: value LED -> Pwr_L.E.D
- D2: value DIODE -> Pwr; moved to F.Cu
- J3, J5: footprint Pin_Headers:Pin_Header_Straight_1x02_Pitch2.54mm -> Custom_Libraries:Battery_holder
- SW2: value SW_Push -> On/Off
- U5: value Select_IN -> Slide_switch
- moved J4 16.9 mm to (41.5, 20.4)
- moved D2 16.2 mm to (48.0, 54.8), turned to 90 degrees
- moved J3 14.9 mm to (40.4, 56.3), turned to 0 degrees
- moved C6 14.5 mm to (46.5, 59.5)
- moved D1 12.8 mm to (45.2, 41.7)
- moved SW2 9.73 mm to (38.7, 47.1)
- moved U3 9.63 mm to (57.1, 58.0)
- moved R5 8.60 mm to (58.1, 20.7)
- moved J5 7.93 mm to (32.2, 56.4), turned to 0 degrees
- moved R3 7.58 mm to (41.9, 42.4)
- moved C2 5.39 mm to (34.4, 29.4)
- moved C3 4.52 mm to (45.4, 35.1)
- moved C4 4.52 mm to (47.9, 35.1)
- moved R2 4.52 mm to (49.9, 35.1)
- moved U2 4.52 mm to (46.9, 34.6)
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Connections:
- net /DSW_1 renamed Net-(U2-Pad33)
- net /DSW_2 renamed Net-(U2-Pad32)
- net /DSW_3 renamed Net-(U2-Pad21)
- net /DSW_4 renamed Net-(U2-Pad22)
- net /Reset renamed /Reset_LoRa
- net Net-(U2-Pad39) renamed /EchoToStm
- C6 pad 2: /BAT_+ve -> /BAT_IN
- D1 pad 1: /BAT_+ve -> Net-(D1-Pad1)
- D1 pad 2: Net-(D1-Pad2) -> /Slide
- R3 pad 1: Net-(D1-Pad2) -> Net-(D1-Pad1)
- SW2 pad 1: /BAT_IN -> /Slide
- SW2 pad 2: /BAT_+ve -> /VCC3V3
- U1 pad 1: /BAT_+ve -> /BAT_IN
- U1 pad 3: /BAT_+ve -> /BAT_IN
- U2 pad 40: Net-(U2-Pad40) -> /Trig
- U5 pad 1: /BAT_+ve -> /BAT_IN
- U5 pad 2: /VCC3V3 -> /Slide
- U5 pad 5: /VCC3V3 -> /Slide
- U5 pad 6: /BAT_+ve -> /BAT_IN
Routing:
- net GNDREF: track 199.9 -> 0.00 mm, vias 2 -> 0
- net /VCC3V3: track 165.4 -> 0.00 mm
- net /RESET: track 83.8 -> 0.00 mm, vias 8 -> 0
- net /OSCIN: track 60.6 -> 0.00 mm
- net /OSCOUT: track 49.4 -> 0.00 mm
- net /SDA: track 42.8 -> 0.00 mm, vias 1 -> 0
- net /SCL: track 38.9 -> 0.00 mm, vias 1 -> 0
- net /BAT_+ve: track 35.7 -> 0.00 mm
- net /Reset_LoRa: track 29.9 -> 0.00 mm, vias 1 -> 0
- net /DIO0: track 24.4 -> 0.00 mm, vias 1 -> 0
- net /PC15: track 23.5 -> 0.00 mm
- net /Supply_Reg: track 23.5 -> 0.00 mm
- net /DIO1: track 20.8 -> 0.00 mm, vias 1 -> 0
- net /RX0: track 20.6 -> 0.00 mm
- net /LDR_IN: track 19.2 -> 0.00 mm, vias 1 -> 0
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Other:
- board text added: "Hukam Technologies"
- board text added: "Sensor_PCB_v1"

Commit message: update
Parts:
- D1: value Pwr_L.E.D -> Pwr; moved to F.Cu
- D2: value Pwr -> DIODE; moved to B.Cu
- J1: value Header 3x2 -> Boot
- J6: value Distance / -> Distance
- SW2: value On/Off -> On / Off
- U1: moved to B.Cu
- moved J6 35.3 mm to (24.9, 32.7)
- moved D1 13.1 mm to (47.5, 54.6)
- moved U4 3.86 mm to (33.2, 34.9)
- moved D2 3.80 mm to (45.2, 57.4), turned to 270 degrees
- moved C6 1.70 mm to (47.6, 60.7), turned to 270 degrees
- moved J1 1.34 mm to (60.4, 25.9)
- moved J2 0.81 mm to (65.8, 33.3)
- moved U3 0.61 mm to (57.4, 57.5)
- moved C7 0.36 mm to (30.6, 43.0)
- turned U1 to 270 degrees
Connections:
- net /Touch_1 renamed Net-(U2-Pad10)
- net /Touch_2 renamed Net-(U2-Pad25)
- U2 pad 2: /Touch_3 -> Net-(U2-Pad2)
- U2 pad 26: /Touch_3 -> Net-(U2-Pad26)
Routing:
- net GNDREF: track 0.00 -> 254.2 mm
- net /VCC3V3: track 0.00 -> 155.5 mm
- net /LDR_IN: track 0.00 -> 58.7 mm
- net /Trig: track 0.00 -> 45.4 mm
- net /SWIO: track 0.00 -> 41.2 mm
- net /SCL: track 0.00 -> 40.5 mm
- net /PC14: track 0.00 -> 38.6 mm
- net /BAT_IN: track 0.00 -> 38.3 mm
- net /Echo: track 0.00 -> 37.1 mm, vias 0 -> 1
- net /SDA: track 0.00 -> 35.0 mm
- net /Slide: track 0.00 -> 32.8 mm
- net /Reset_LoRa: track 0.00 -> 31.6 mm, vias 0 -> 1
- net /DIO0: track 0.00 -> 29.1 mm, vias 0 -> 1
- net /OSCOUT: track 0.00 -> 28.8 mm, vias 0 -> 1
- net /OSCIN: track 0.00 -> 28.0 mm, vias 0 -> 1
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Other:
- board outline added: 46 x 44 mm
- rule trace_min: 0.2 -> 0.3
- rule via_min_size: 0.4 -> 4.5

Commit message: update
Parts:
- AE1: value ANT -> Antenna
- D1: value Pwr -> Pwr_L.E.D
- J1: value Boot -> Header 3x2
- J6: value Distance -> Distance /
- SW1: footprint Buttons_Switches_SMD:SW_DIP_x1_W7.62mm_Slide_Copal_CHS-B -> Buttons_Switches_SMD:SW_SPST_B3U-1000P
- SW2: value On / Off -> SW_Push
- moved SW1 18.8 mm to (57.7, 37.0), turned to 180 degrees
- moved J2 0.83 mm to (65.0, 33.1)
Connections:
- C1 pad 1: GNDREF -> Net-(C1-Pad1)
- C2 pad 2: GNDREF -> GND
- C3 pad 2: GNDREF -> GND
- C4 pad 2: GNDREF -> GND
- C5 pad 2: GNDREF -> GND
- C6 pad 1: GNDREF -> GND
- C7 pad 1: GNDREF -> GND
- J1 pad 3: GNDREF -> GND
- J1 pad 4: /VCC3V3 -> GND
- J1 pad 6: GNDREF -> /VCC3V3
- J2 pad 5: GNDREF -> GND
- J3 pad 1: GNDREF -> GND
- J4 pad 1: GNDREF -> GND
- J5 pad 1: GNDREF -> GND
- J6 pad 1: GNDREF -> GND
- R3 pad 2: GNDREF -> GND
- R5 pad 2: GNDREF -> GND
- R7 pad 1: GNDREF -> GND
- SW1 pad 1: GNDREF -> GND
- U1 pad 2: GNDREF -> GND
- U2 pad 23: GNDREF -> GND
- U2 pad 35: GNDREF -> GND
- U2 pad 47: GNDREF -> GND
- U2 pad 8: GNDREF -> GND
- U3 pad 16: GNDREF -> GND
- U3 pad 2: GNDREF -> GND
- U3 pad 9: GNDREF -> GND
- U4 pad 2: GNDREF -> GND
Routing:
- net GNDREF: track 254.2 -> 0.00 mm
- net GND: track 0.00 -> 205.7 mm, vias 0 -> 21
- net /OSCOUT: track 28.8 -> 73.6 mm, vias 1 -> 0
- net /OSCIN: track 28.0 -> 50.9 mm, vias 1 -> 0
- net /SWIO: track 41.2 -> 19.3 mm
- net /Echo: track 37.1 -> 58.1 mm, vias 1 -> 0
- net /BOOT1: track 18.4 -> 38.1 mm, vias 1 -> 0
- net /BOOT0: track 12.6 -> 28.4 mm, vias 0 -> 3
- net /RESET: track 17.6 -> 33.0 mm, vias 1 -> 2
- net /Trig: track 45.4 -> 57.9 mm, vias 0 -> 2
- net /PC14: track 38.6 -> 26.7 mm
- net /SCL: track 40.5 -> 28.6 mm
- net /VCC3V3: track 155.5 -> 167.4 mm, vias 0 -> 5
- net /SDA: track 35.0 -> 44.2 mm
- net /RX0: track 14.7 -> 21.6 mm
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- added copper zone on B.Cu, net GND
- added copper zone on F.Cu, net GND
Other:
- net class Default: clearance 0.2 -> 0.25
- rule trace_clearance: 0.2 -> 0.25
- rule trace_min: 0.3 -> 0.25
- rule via_min_size: 4.5 -> 0.25
- board text added: "+ve"
- board text added: "-ve"
- board text added: "3.3 V"
- board text added: "3.3V"
- board text added: "5V"
- board text added: "BOOT0"
- board text added: "BOOT1"
- board text added: "Battery"
- board text added: "Battery_In"
- board text added: "Distance"
- board text added: "Echo"
- board text added: "GND"
- board text added: "ON/OFF"
- board text added: "Power"
- board text added: "Prog_Hdr"
- board text added: "Reg_Supply"
- board text added: "Reset"
- board text added: "Rx"
- board text added: "SCL"
- board text added: "SDA"
- board text added: "SWCLK"
- board text added: "SWIO"
- board text added: "Solar"
- board text added: "Stm32"
- board text added: "Trig"
- board text added: "Tx"
