File: Designs/PCB/KiCad/Projects/SwitchBoard/Sensor_pcb/Sensor_all/Sensor_pcb_v1/Sensor_pcb_v1.sch (KiCad schematic (older format))
At the start: 25 parts, among them J1 Header 3x2, J2 Prog Hdr, J3 Header_In, J4 SWD, SW1 SW_Push, U1 APK2112.K-3.3, U2 STM32, U3 LoRa, Y1 32.768K, Y2 8Mhz

Commit message: update
Parts:
- removed J3: Header_In, Pin_Headers:Pin_Header_Straight_1x08_Pitch2.54mm, symbol Connector:Conn_01x08_Female
- added R4: 10K, Resistors_SMD:R_0805, symbol Device:R
- added R5: LDR, Diodes_THT:D_A-405_P5.08mm_Vertical_AnodeUp, symbol Sensor_Optical:LDR03
- added SW2: SW_Push, Buttons_Switches_THT:SW_PUSH_6mm_h5mm, symbol Switch:SW_Push
- added U4: BME_280, Custom_Libraries:BME280, symbol Sensor_Humidity:BME_280
- added U5: Slide_switch, Buttons_Switches_THT:SW_DIP_x3_W7.62mm_Slide_LowProfile, symbol Switch:Slide_switch
- C1: value 105 -> 1.0uf
- D2: renamed from D?; footprint (none) -> Diodes_SMD:D_0805
- J3, J5: renamed from J?; footprint (none) -> Pin_Headers:Pin_Header_Straight_1x02_Pitch2.54mm
Connections:
- net BAT_+ve: now also C6.2, D1.1 (K), U1.1 (VIN), U1.3 (EN), SW2.2, U5.1, U5.6
- net GNDREF: now also R5.2, U4.2 (GND)
- net VCC3V3: now also R4.2, U4.1 (VSS), U5.2, U5.5; no longer C7.2, D1.1 (K), U1.5 (VOUT)
- net SCL: now reaches U2.45 (PB8)
- net SCL: now also U4.3 (SCL)
- net SDA: now reaches U2.46 (PB9)
- net SDA: now also U4.4 (SDA)
- net BAT_IN: now reaches D2.2 (K), J5.2 (Pin_2)
- net BAT_IN: now also SW2.1
- removed net +5V: C6.2, J2.4 (Pin_4), U1.1 (VIN), U1.3 (EN)
- net Opto_IN renamed LDR_IN
- net LDR_IN: now also R4.1, R5.1
- new net 5V: J2.4 (Pin_4)
- new net Supply_Reg: C7.2, U1.5 (VOUT), U5.3, U5.4
Other:
- note added: "Crystals for Clock\n"
- note added: "STM32FXXX\n"
- note removed: "Input / Output Headers"
- note removed: "STM & Crystals\n"
- moved on the sheet: AE1, C1, C2, C3, C4, C5, C6, C7, D1, D2, J1, J2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

Commit message: Update
Parts:
- added J6: Distance /, Pin_Headers:Pin_Header_Straight_1x04_Pitch2.54mm, symbol Connector:Conn_01x04_Female
- added R6: 2.7K, Resistors_SMD:R_0805, symbol Device:R
- added R7: 4.7K, Resistors_SMD:R_0805, symbol Device:R
- AE1: footprint SMD_Packages:1Pin -> Pin_Headers:Pin_Header_Straight_1x01_Pitch2.54mm
- D1: value LED -> Pwr_L.E.D
- J3, J5: footprint Pin_Headers:Pin_Header_Straight_1x02_Pitch2.54mm -> Custom_Libraries:Battery_holder
Connections:
- net BAT_IN: now also C6.2, U1.1 (VIN), U1.3 (EN), U5.1, U5.6; no longer SW2.1
- net GNDREF: now also J6.1 (Pin_1), R7.1
- net VCC3V3: now also SW2.2, J6.4 (Pin_4); no longer U5.2, U5.5
- net EchoToStm: now reaches U2.39 (PB3)
- net Trig: now reaches U2.40 (PB4)
- net Trig: now also J6.3 (Pin_3)
- net at R3.1: now also D1.1 (K); no longer D1.2 (A)
- removed net BAT_+ve: C6.2, D1.1 (K), SW2.2, U1.1 (VIN), U1.3 (EN), U5.1, U5.6
- net DSW_1: no longer names the net of U2.33 (PA12)
- net DSW_2: no longer names the net of U2.32 (PA11)
- net DSW_3: no longer names the net of U2.21 (PB10)
- net DSW_4: no longer names the net of U2.22 (PB11)
- net Reset renamed Reset_LoRa
- new net Echo: J6.2 (Pin_2), R6.2
- new net EchoToStm32: R6.1, R7.2
- new net Slide: D1.2 (A), SW2.1, U5.2, U5.5
- no-connect marks 8 -> 16
Other:
- note added: "Ultra Sonic"
- moved on the sheet: D1, R3, SW2, U5

Commit message: update
Parts:
- SW1: footprint Buttons_Switches_SMD:SW_DIP_x1_W7.62mm_Slide_Copal_CHS-B -> Buttons_Switches_SMD:SW_SPST_B3U-1000P
Connections:
- net GNDREF renamed GND
- net GND: no longer C1.1
- net Touch_1: no longer names the net of U2.10 (PA0)
- net Touch_2: no longer names the net of U2.25 (PB12)
- net Touch_3: no longer names the net of U2.2 (PC13)
- net Touch_3: no longer U2.26 (PB13)
- no-connect marks 16 -> 20
Changed lines of the file:
@@
 	1143 2244 1143 2544
 Wire Wire Line
-	1143 2544 1343 2544
-Wire Wire Line
-	1343 2544 1743 2544
-Wire Wire Line
 	1743 2544 1743 2244
-Connection ~ 1343 2544
 Text Label 1993 2144 2    50   ~ 0
 BOOT1
@@
 F 0 "SW1" V 2393 2244 50  0000 R CNN
 F 1 "SW_Push" V 2293 2744 50  0001 R CNN
-F 2 "Buttons_Switches_SMD:SW_DIP_x1_W7.62mm_Slide_Copal_CHS-B" H 2393 2494 50  0001 C CNN
+F 2 "Buttons_Switches_SMD:SW_SPST_B3U-1000P" H 2393 2494 50  0001 C CNN
 F 3 "~" H 2393 2494 50  0001 C CNN
 	1    2393 2294
@@
 Wire Wire Line
 	2393 2094 2693 2094
-$Comp
-L power:GNDREF #PWR04
-U 1 1 5F102D01
-P 1343 2544
-F 0 "#PWR04" H 1348 2371 50  0001 C CNN
-F 1 "GNDREF" H 1348 2371 50  0000 C CNN
-F 2 "" H 1343 2544 50  0001 C CNN
-F 3 "" H 1343 2544 50  0001 C CNN
-	1    1343 2544
-	1    0    0    -1
-$EndComp
-Wire Wire Line
-	2393 2494 2693 2494
-Wire Wire Line
-	2793 2494 2793 2544
 $Comp
 L Device:C C1
@@
 Wire Wire Line
 	2693 2444 2693 2494
-Connection ~ 2693 2494
-Wire Wire Line
-	2693 2494 2793 2494
 Wire Wire Line
 	2693 2144 2693 2094
@@
 	2693 1994 2693 2094
 $Comp
-L power:GNDREF #PWR02
-U 1 1 5F1282A4
-P 2793 2544
-F 0 "#PWR02" H 2798 2371 50  0001 C CNN
-F 1 "GNDREF" H 2798 2371 50  0000 C CNN
-F 2 "" H 2793 2544 50  0001 C CNN
-F 3 "" H 2793 2544 50  0001 C CNN
-	1    2793 2544
-	1    0    0    -1
-$EndComp
-$Comp
 L Regulator_Linear:AP2112K-3.3 U1
 U 1 1 5F13570F
@@
 Connection ~ 2375 4852
 $Comp
-L power:GNDREF #PWR03
+L power:GND #PWR03
 U 1 1 5F13CA0F
 P 2675 5302
 F 0 "#PWR03" H 2680 5129 50  0001 C CNN
-F 1 "GNDREF" H 2680 5129 50  0000 C CNN
+F 1 "GND" H 2680 5129 50  0000 C CNN
 F 2 "" H 2675 5302 50  0001 C CNN
 F 3 "" H 2675 5302 50  0001 C CNN
@@
 GND
 Connection ~ 2675 5252
-$Comp
-L Connector_Generic:Conn_01x05 J2
-U 1 1 5F0DE12E
-P 10269 5607
-F 0 "J2" H 10187 5182 50  0000 C CNN
-F 1 "Prog Hdr" H 10187 5273 50  0000 C CNN
-F 2 "Pin_Headers:Pin_Header_Straight_1x05_Pitch2.54mm" H 10269 5607 50  0001 C CNN
-F 3 "~" H 10269 5607 50  0001 C CNN
-	1    10269 5607
-	-1   0    0    1
-$EndComp
 Text Label 10669 5407 2    50   ~ 0
 GND
@@
 Text Label 2993 2494 0    50   ~ 0
 GND
-Wire Wire Line
-	2793 2494 2993 2494
-Connection ~ 2793 2494
 Text Label 1893 2544 0    50   ~ 0
 GND
@@
 Text Notes 9556 4199 0    50   Italic 0
 Sensors\n
-Text Label 4364 2290 0    50   ~ 0
-Touch_1
-Text Label 4364 1490 0    50   ~ 0
-Touch_3
 NoConn ~ 4664 1390
 Text Notes 9768 2065 0    50   Italic 0
@@
 Text Label 5914 3290 1    50   ~ 0
 BOOT1
-Text Label 7214 2390 2    50   ~ 0
-Touch_3
 Wire Wire Line
 	5414 3290 5414 2990
@@
 Wire Wire Line
 	5914 2990 5914 3290
-Text Label 7214 2490 2    50   ~ 0
-Touch_2
 Wire Wire Line
 	5214 3290 5214 2990
@@
 	2550 7280 2800 7280
 Connection ~ 2550 7080
-NoConn ~ 6870 1690
-NoConn ~ 6870 1790
 Wire Wire Line
 	4414 2490 4664 2490
 Wire Wire Line
-	4364 2290 4664 2290
-Wire Wire Line
 	4314 2190 4664 2190
 Wire Wire Line
@@
 	4664 1590 4364 1590
 Wire Wire Line
-	4364 1490 4664 1490
-Wire Wire Line
 	6864 1390 7264 1390
 Wire Wire Line
-	7214 2390 6864 2390
-Wire Wire Line
 	7164 1490 6864 1490
-Wire Wire Line
-	6864 2490 7214 2490
 Wire Wire Line
 	6864 1590 7214 1590
@@
 Wire Wire Line
 	2175 4852 2375 4852
+NoConn ~ 6864 2490
+NoConn ~ 6864 2390
+NoConn ~ 6864 1690
+NoConn ~ 6864 1790
+NoConn ~ 4664 2290
+NoConn ~ 4664 1490
+$Comp
+L Connector_Generic:Conn_01x05 J2
+U 1 1 5F0DE12E
+P 10269 5607
+F 0 "J2" H 10187 5182 50  0000 C CNN
+F 1 "Prog Hdr" H 10244 5934 50  0000 C CNN
+F 2 "Pin_Headers:Pin_Header_Straight_1x05_Pitch2.54mm" H 10269 5607 50  0001 C CNN
+F 3 "~" H 10269 5607 50  0001 C CNN
+	1    10269 5607
+	-1   0    0    1
+$EndComp
+$Comp
+L power:GND #PWR?
+U 1 1 5F1737D3
+P 1741 2632
+F 0 "#PWR?" H 1746 2459 50  0001 C CNN
+F 1 "GND" H 1746 2459 50  0000 C CNN
+F 2 "" H 1741 2632 50  0001 C CNN
+F 3 "" H 1741 2632 50  0001 C CNN
+	1    1741 2632
+	1    0    0    -1
+$EndComp
+Wire Wire Line
+	1143 2544 1743 2544
+Wire Wire Line
+	1743 2543 1741 2632
+$Comp
+L power:GND #PWR?
+U 1 1 5F17DC84
+P 2695 2607
+F 0 "#PWR?" H 2700 2434 50  0001 C CNN
+F 1 "GND" H 2700 2434 50  0000 C CNN
+F 2 "" H 2695 2607 50  0001 C CNN
+F 3 "" H 2695 2607 50  0001 C CNN
+	1    2695 2607
+	1    0    0    -1
+$EndComp
+Wire Wire Line
+	2393 2494 2695 2494
+Wire Wire Line
+	2695 2607 2695 2494
+Connection ~ 2695 2494
+Wire Wire Line
+	2695 2494 2993 2494
 $EndSCHEMATC
