File: Designs/PCB/KiCad/Projects/SwitchBoard/Sensor_pcb/Sensor_PCB_v3/Sensor_pcb_v3.sch (KiCad schematic (older format))
At the start: 42 parts, among them J1 Solar_input, J2 Battery_input, J3 Distance /, J4 SWD, J5 Airquality, Q1 BC547, SW1 MLL1200S, SW2 SW_Push, U1 APK2112.K-3.3, U2 LoRa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

Commit message: update
Connections:
- net DIO1: no longer U3.13 (PA3)
- no-connect marks 20 -> 21
Changed lines of the file:
@@
 Wire Wire Line
 	5914 2990 5914 3290
-Wire Wire Line
-	5214 3290 5214 2990
-Text Label 5214 3290 1    50   ~ 0
-DIO1
 Text Label 5414 3290 1    50   ~ 0
 SCK
@@
 	3247 2714 3435 2714
 Connection ~ 3247 2714
+NoConn ~ 5214 2990
 $EndSCHEMATC

Commit message: Update
Parts:
- removed C? (x2): 100 uF, Custom_Libraries:CAPAE660X550N, symbol capacitor_electolytic:ECA-1EM102
- removed C? (x2): 1 uf, Capacitors_SMD:C_0805, symbol Device:C
- removed D?: 1N5817, Diodes_SMD:D_1206, symbol Diode:1N5817
- removed J4: SWD, Pin_Headers:Pin_Header_Straight_1x04_Pitch2.54mm, symbol Connector:Conn_01x04_Female
- removed L?: Inductor_22uH, Custom_Libraries:IND_1248AS-H-220M=P3, symbol 1248AS-H-220M_P3:Inductor_22uH
- removed R6: 2.7K, Resistors_SMD:R_0805, symbol Device:R
- removed R7: 4.7K, Resistors_SMD:R_0805, symbol Device:R
- removed U?: MAX756, Custom_Libraries:SO08, symbol Converter_DCDC:MAX756
- added C8, C9: 100 uF, Custom_Libraries:CAPAE660X550N, symbol capacitor_electolytic:ECA-1EM102
- added D5: SS14, Diodes_SMD:D_1206, symbol Device:D_Zener
- added J4: Conn_01x06_Female, Pin_Headers:Pin_Header_Straight_1x06_Pitch2.54mm, symbol Connector:Conn_01x06_Female
- added L1: Inductor_22uH, Custom_Libraries:IND_1248AS-H-220M=P3, symbol 1248AS-H-220M_P3:Inductor_22uH
- added U5: BL8530, Custom_Libraries:SOT89, symbol Power_Management:BL8530
- Q1: footprint Package_TO_SOT_THT:TO-92_Inline -> Custom_Libraries:BC547-SOT23
Connections:
- net Echo is gone; now on net EchoToStm32: J3.2 (Pin_2)
- net BAT_IN: now also U3.11 (PA1); no longer U3.10 (PA0)
- net DIO0: now also U3.10 (PA0); no longer U3.11 (PA1)
- net GND: now also C8.1, C9.1, J4.1 (Pin_1), U5.1 (GND)
- net OUT_5V: now also C9.2, D5.1 (K), U5.2 (OUT)
- net SWCLK: now also J4.2 (Pin_2)
- net SWIO: now also J4.3 (Pin_3)
- net Supply_Reg: now also C8.2, L1.1
- net VCC3V3: now also J4.6 (Pin_6)
- net TX: now reaches U3.30 (PA9)
- net TX: now also J4.5 (Pin_5)
- net RX: now reaches U3.31 (PA10)
- net RX: now also J4.4 (Pin_4)
- net DIO1: no longer names the net of U3.26 (PB13)
- net DIO1: no longer U2.6 (DIO1)
- net DIO2: no longer names the net of U3.25 (PB12)
- net DIO2: no longer U2.7 (DIO2)
- new net: D5.2 (A), L1.2, U5.3 (LX)
