File: Designs/PCB/KiCad/Projects/SwitchBoard/Sensor_pcb/Sensor_PCB_v3/Sensor_pcb_v3.kicad_pcb (KiCad board)
At the start: 2 copper layers, 35 parts, among them J1 Solar_input, J2 Battery_input, J3 Distance /, J4 SWD, J5 Airquality, Q1 BC547, SW1 MLL1200S, SW2 SW_Push, U1 APK2112.K-3.3, U2 LoRa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

Commit message: Update
Parts:
- removed R6: 2.7K, Resistors_SMD:R_0805
- removed R7: 4.7K, Resistors_SMD:R_0805
- added C8: 100 uF, Custom_Libraries:CAPAE660X550N, F.Cu at (44.1, 32.0)
- added C9: 100 uF, Custom_Libraries:CAPAE660X550N, F.Cu at (73.3, 32.0)
- added D5: SS14, Diodes_SMD:D_1206, F.Cu at (64.2, 34.7)
- added L1: Inductor_22uH, Custom_Libraries:IND_1248AS-H-220M=P3, F.Cu at (54.5, 32.1)
- added U5: BL8530, Custom_Libraries:SOT89, F.Cu at (64.4, 27.9)
- C1, C2, C3, C4, C5, C6, C7, D2, Q1, R1, R2, R3, R4, R8, R9, U1, U2: moved to F.Cu
- J4: value SWD -> Conn_01x06_Female; footprint Pin_Headers:Pin_Header_Straight_1x04_Pitch2.54mm -> Pin_Headers:Pin_Header_Straight_1x06_Pitch2.54mm
- moved AE1 120.9 mm to (25.9, 64.3)
- moved D1 109.4 mm to (36.2, 26.2), turned to 270 degrees
- moved U2 105.6 mm to (34.2, 72.6), turned to 0 degrees
- moved SW1 99.5 mm to (51.3, 21.5), turned to 180 degrees
- moved D2 75.5 mm to (28.2, 34.1), turned to 180 degrees
- moved R1 73.1 mm to (38.8, 21.8), turned to 270 degrees
- moved Y1 72.7 mm to (70.3, 49.8)
- moved R9 72.4 mm to (34.7, 48.6), turned to 270 degrees
- moved U1 71.3 mm to (36.1, 32.0)
- moved J1 70.6 mm to (29.7, 40.0)
- moved C3 70.5 mm to (45.3, 24.3)
- moved J2 70.4 mm to (29.7, 28.4)
- moved C5 69.9 mm to (65.4, 44.6)
- moved D4 69.5 mm to (37.8, 48.6)
- moved C4 69.4 mm to (70.3, 44.6)
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Connections:
- J3 pad 2: /Echo -> /EchoToStm32
- J3 pad 4: /BAT_IN -> /OUT_5V
- J4 pad 4: /VCC3V3 -> /RX
- Q1 pad 1: /Solar_+ve -> /Charge
- Q1 pad 2: /Charge -> Net-(D2-Pad1)
- Q1 pad 3: Net-(D2-Pad1) -> /Solar_+ve
- U2 pad 6: /DIO1 -> Net-(U2-Pad6)
- U3 pad 10: /BAT_IN -> /DIO0
- U3 pad 11: /Reset_LoRa -> /BAT_IN
- U3 pad 12: /DIO0 -> Net-(U3-Pad12)
- U3 pad 13: /DIO1 -> Net-(U3-Pad13)
- U3 pad 2: Net-(U3-Pad2) -> /Reset_LoRa
- U3 pad 30: Net-(U3-Pad30) -> /TX
- U3 pad 31: Net-(U3-Pad31) -> /RX
Routing:
- net (no net): vias 0 -> 4
- removed copper zone on B.Cu, net /GND
- removed copper zone on F.Cu, net /GND
Other:
- board text added: "Charging"
- board text added: "LDR"
- board text added: "RX"
- board text added: "Sensor_PCB_v3"
- board text added: "TX"
- board text removed: "Sensor_PCB_v2"

Commit message: update
Parts:
- added M1: MountingHole_1.5mm, Custom_Libraries:MountingHole1.5mm, F.Cu at (25.4, 21.4)
- added M2: MountingHole_1.5mm, Custom_Libraries:MountingHole1.5mm, F.Cu at (25.4, 87.8)
- added M2: MountingHole_1.5mm, Custom_Libraries:MountingHole1.5mm, F.Cu at (58.2, 21.4)
- added M3: MountingHole_1.5mm, Custom_Libraries:MountingHole1.5mm, F.Cu at (58.2, 87.8)
- C1, C2, C3, C4, C5, C6, C7, D2, D5, Q1, R1, R2, R3, R4, R8, R9, U1, U3, U5: moved to B.Cu
- moved U4 42.9 mm to (50.0, 65.8)
- moved C2 38.2 mm to (46.4, 77.4), turned to 180 degrees
- moved J4 36.7 mm to (37.7, 86.7)
- moved R2 36.6 mm to (47.9, 73.4), turned to 180 degrees
- moved R8 34.9 mm to (25.6, 63.0), turned to 270 degrees
- moved R4 34.3 mm to (52.0, 26.2)
- moved J3 34.0 mm to (55.5, 47.5)
- moved R5 33.4 mm to (57.6, 26.3), turned to 120 degrees
- moved J5 33.1 mm to (56.2, 80.5)
- moved SW2 29.7 mm to (51.1, 79.6)
- moved C4 28.2 mm to (42.2, 47.9), turned to 90 degrees
- moved Y2 26.5 mm to (26.7, 47.9), turned to 270 degrees
- moved C5 24.2 mm to (42.3, 51.8), turned to 90 degrees
- moved Y1 23.9 mm to (46.5, 48.0), turned to 270 degrees
- moved AE1 23.6 mm to (28.6, 87.7)
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Routing:
- net /GND: track 0.00 -> 347.9 mm
- net /VCC3V3: track 0.00 -> 235.7 mm, vias 0 -> 1
- net /EchoToStm32: track 0.00 -> 89.3 mm
- net /LDR_IN: track 0.00 -> 82.6 mm
- net /BAT_IN: track 0.00 -> 70.2 mm
- net /SWCLK: track 0.00 -> 64.3 mm, vias 0 -> 1
- net /RX: track 0.00 -> 63.8 mm, vias 0 -> 1
- net /TX: track 0.00 -> 56.1 mm, vias 0 -> 1
- net /OUT_5V: track 0.00 -> 49.0 mm
- net /SWIO: track 0.00 -> 37.0 mm
- net /Air_in: track 0.00 -> 33.9 mm, vias 0 -> 1
- net /OSCIN: track 0.00 -> 33.5 mm, vias 0 -> 1
- net /Supply_Reg: track 0.00 -> 32.9 mm, vias 0 -> 1
- net /Charge: track 0.00 -> 29.2 mm, vias 0 -> 2
- net Net-(D3-Pad2): track 0.00 -> 29.0 mm, vias 0 -> 1
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- added copper zone on B.Cu, net /GND
- added copper zone on F.Cu, net /GND
Other:
- net class Antenna added: clearance 0.2, trace_width 0.8, via_dia 1, via_drill 0.6
- net class Default: trace_width 0.17 -> 0.2
- board text removed: "Distance"
