File: Designs/PCB/KiCad/Projects/SwitchBoard/Sensor_pcb/Sensor_PCB_v4/Sensor_pcb_v4.kicad_pcb (KiCad board)
At the start: 2 copper layers, 50 parts, among them IC1 TP4056, J1 Solar_input, J2 Battery_input, J3 Distance /, J4 Conn_01x06_Female, J5 Airquality, J6 USB3130-XX-X_REVD, M1 MountingHole_2.1mm, M2 MountingHole_2.1mm, M3 MountingHole_2.1mm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

Commit message: learnings
Changed lines of the file:
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@@
-(kicad_pcb (version 20171130) (host pcbnew 5.1.6-c6e7f7d~87~ubuntu18.04.1)
+(kicad_pcb (version 20171130) (host pcbnew 5.1.7-a382d34a8~88~ubuntu18.04.1)
   (general
     (thickness 1.6)
@@
     (visible_elements FFFFFF7F)
     (pcbplotparams
-      (layerselection 0x3f1ff_ffffffff)
-      (usegerberextensions false)
+      (layerselection 0x3ffff_ffffffff)
+      (usegerberextensions true)
       (usegerberattributes false)
       (usegerberadvancedattributes false)
@@
       (effects (font (size 1 1) (thickness 0.15)))
     )
-    (fp_text value BME_280 (at -1.06138 -1.29286 90) (layer Dwgs.User)
+    (fp_text value BME_280 (at -1.06138 -1.29286 90) (layer F.SilkS)
       (effects (font (size 1 1) (thickness 0.15)))
     )
@@
     (tags "capacitor 0805")
     (attr smd)
-    (fp_text reference C10 (at 0 -1.5) (layer Dwgs.User)
+    (fp_text reference C10 (at 0 -1.5) (layer F.SilkS)
       (effects (font (size 1 1) (thickness 0.15)))
     )
@@
     (tags "smd diode")
     (attr smd)
-    (fp_text reference D3 (at -2.63652 0.23368) (layer Dwgs.User)
+    (fp_text reference D3 (at -2.63652 0.23368) (layer F.SilkS)
       (effects (font (size 1 1) (thickness 0.15)))
     )
@@
     (tags "smd diode")
     (attr smd)
-    (fp_text reference D6 (at -1.21158 -1.57988) (layer Dwgs.User)
+    (fp_text reference D6 (at -1.21158 -1.57988) (layer F.SilkS)
       (effects (font (size 1 1) (thickness 0.15)))
     )
@@
     (tags SOT-23)
     (attr smd)
-    (fp_text reference Q1 (at 2.3622 0.09144 180) (layer Dwgs.User)
+    (fp_text reference Q1 (at 2.3622 0.09144 180) (layer F.SilkS)
       (effects (font (size 1 1) (thickness 0.15)))
     )
@@
     (tags "resistor 0805")
     (attr smd)
-    (fp_text reference R8 (at -2.4638 -0.43942) (layer Dwgs.User)
+    (fp_text reference R8 (at -2.4638 -0.43942) (layer F.SilkS)
       (effects (font (size 1 1) (thickness 0.15)))
     )
@@
     (tags "resistor 0805")
     (attr smd)
-    (fp_text reference R10 (at -0.3683 -1.4351) (layer Dwgs.User)
+    (fp_text reference R10 (at -0.3683 -1.4351) (layer F.SilkS)
       (effects (font (size 1 1) (thickness 0.15)))
     )
@@
     )
   )
-  (gr_text 5V (at 58.18632 55.20436) (layer Dwgs.User)
+  (gr_text 5V (at 58.18632 55.20436) (layer F.SilkS)
     (effects (font (size 0.7 0.7) (thickness 0.1)))
   )
-  (gr_text Trig (at 58.3057 52.50942) (layer Dwgs.User)
+  (gr_text Trig (at 58.3057 52.50942) (layer F.SilkS)
     (effects (font (size 0.7 0.7) (thickness 0.1)))
   )
-  (gr_text Echo (at 58.46318 49.80178) (layer Dwgs.User)
+  (gr_text Echo (at 58.46318 49.80178) (layer F.SilkS)
     (effects (font (size 0.7 0.7) (thickness 0.1)))
   )
-  (gr_text 3.3V (at 59.15914 80.15224) (layer Dwgs.User)
+  (gr_text 3.3V (at 59.15914 80.15224) (layer F.SilkS)
     (effects (font (size 0.7 0.7) (thickness 0.1)))
   )
-  (gr_text GND (at 59.04992 77.56398) (layer Dwgs.User)
+  (gr_text GND (at 59.04992 77.56398) (layer F.SilkS)
     (effects (font (size 0.7 0.7) (thickness 0.1)))
   )
@@
     (arrow2b (pts (xy 23.308317 90.812618) (xy 24.435393 90.227298)))
   )
-  (gr_text RX (at 43.3959 89.0524 270) (layer Dwgs.User)
+  (gr_text RX (at 43.3959 89.0524 270) (layer F.SilkS)
     (effects (font (size 0.5 0.5) (thickness 0.08)))
   )
-  (gr_text TX (at 45.91304 88.84158 270) (layer Dwgs.User)
+  (gr_text TX (at 45.91304 88.84158 270) (layer F.SilkS)
     (effects (font (size 0.5 0.5) (thickness 0.08)))
   )
-  (gr_text LDR (at 52.6542 24.3713) (layer Dwgs.User)
+  (gr_text LDR (at 52.6542 24.3713) (layer F.SilkS)
     (effects (font (size 0.8 0.8) (thickness 0.1)))
   )
-  (gr_text +ve (at 24.8031 43.15206 270) (layer Dwgs.User)
+  (gr_text +ve (at 24.8031 43.15206 270) (layer F.SilkS)
     (effects (font (size 1 1) (thickness 0.1)))
   )
-  (gr_text -ve (at 24.74722 36.67506 270) (layer Dwgs.User)
+  (gr_text -ve (at 24.74722 36.67506 270) (layer F.SilkS)
     (effects (font (size 1 1) (thickness 0.1)))
   )
-  (gr_text Solar (at 23.9903 40.13708 270) (layer Dwgs.User)
+  (gr_text Solar (at 23.9903 40.13708 270) (layer F.SilkS)
     (effects (font (size 1 1) (thickness 0.15)))
   )
-  (gr_text +ve (at 24.83104 32.55772 270) (layer Dwgs.User)
+  (gr_text +ve (at 24.83104 32.55772 270) (layer F.SilkS)
     (effects (font (size 1 1) (thickness 0.1)))
   )
@@
     (effects (font (size 1 1) (thickness 0.15)))
   )
-  (gr_text GND (at 35.5854 88.84158 270) (layer Dwgs.User)
+  (gr_text GND (at 35.5854 88.84158 270) (layer F.SilkS)
     (effects (font (size 0.5 0.5) (thickness 0.08)))
   )
-  (gr_text CLK (at 38.24224 89.11082 270) (layer Dwgs.User)
+  (gr_text CLK (at 38.24224 89.11082 270) (layer F.SilkS)
     (effects (font (size 0.5 0.5) (thickness 0.08)))
   )
-  (gr_text IO (at 40.82034 88.9635 270) (layer Dwgs.User)
+  (gr_text IO (at 40.82034 88.9635 270) (layer F.SilkS)
     (effects (font (size 0.5 0.5) (thickness 0.08)))
   )
-  (gr_text vcc (at 48.51146 89.04986 270) (layer Dwgs.User)
+  (gr_text vcc (at 48.51146 89.04986 270) (layer F.SilkS)
     (effects (font (size 0.5 0.5) (thickness 0.08)))
   )
   (gr_line (start 93.93682 48.25238) (end 93.94952 48.22698) (layer Margin) (width 0.15))
   (gr_line (start 93.93682 48.23968) (end 93.93682 48.25238) (layer Margin) (width 0.15))
-  (gr_text On (at 41.148 20.45462) (layer Dwgs.User)
+  (gr_text On (at 41.148 20.45462) (layer F.SilkS)
     (effects (font (size 1 1) (thickness 0.2)))
   )
-  (gr_text Off (at 52.67452 20.57654) (layer Dwgs.User)
+  (gr_text Off (at 52.67452 20.57654) (layer F.SilkS)
     (effects (font (size 1 1) (thickness 0.2)))
   )
-  (gr_text -ve (at 24.74722 24.4094 270) (layer Dwgs.User)
+  (gr_text -ve (at 24.74722 24.4094 270) (layer F.SilkS)
     (effects (font (size 1 1) (thickness 0.1)))
   )
-  (gr_text "3.3 V" (at 57.66562 68.70446) (layer Dwgs.User)
+  (gr_text "3.3 V" (at 57.66562 68.70446) (layer F.SilkS)
     (effects (font (size 0.7 0.7) (thickness 0.1)))
   )
-  (gr_text GND (at 57.40908 66.02984) (layer Dwgs.User)
+  (gr_text GND (at 57.40908 66.02984) (layer F.SilkS)
     (effects (font (size 0.7 0.7) (thickness 0.1)))
   )
-  (gr_text SCL (at 57.37098 63.38824) (layer Dwgs.User)
+  (gr_text SCL (at 57.37098 63.38824) (layer F.SilkS)
     (effects (font (size 0.7 0.7) (thickness 0.1)))
   )
-  (gr_text SDA (at 57.33542 60.67552) (layer Dwgs.User)
+  (gr_text SDA (at 57.33542 60.67552) (layer F.SilkS)
     (effects (font (size 0.7 0.7) (thickness 0.1)))
   )
-  (gr_text GND (at 58.24982 47.68596) (layer Dwgs.User)
+  (gr_text GND (at 58.24982 47.68596) (layer F.SilkS)
     (effects (font (size 0.7 0.7) (thickness 0.1)))
   )
-  (gr_text Battery (at 24.12238 28.90012 270) (layer Dwgs.User)
+  (gr_text Battery (at 24.12238 28.90012 270) (layer F.SilkS)
     (effects (font (size 1 1) (thickness 0.15)))
   )
-  (gr_text Reset (at 47.39386 81.74228) (layer Dwgs.User)
+  (gr_text Reset (at 47.39386 81.74228) (layer F.SilkS)
     (effects (font (size 1 1) (thickness 0.15)))
   )
@@
     (effects (font (size 0.8 0.8) (thickness 0.1)))
   )
-  (gr_text Power (at 34.51098 26.31948 270) (layer Dwgs.User)
+  (gr_text Power (at 34.51098 26.31948 270) (layer F.SilkS)
     (effects (font (size 1 1) (thickness 0.15)))
   )
-  (gr_text Sensor_PCB_v4 (at 36.1188 66.22542) (layer Dwgs.User)
+  (gr_text Sensor_PCB_v4 (at 36.1188 66.22542) (layer F.SilkS)
     (effects (font (size 0.6 0.6) (thickness 0.15)))
   )
-  (gr_text "Hukam Technologies\n" (at 35.7251 65.0748) (layer Dwgs.User)
+  (gr_text "Hukam Technologies\n" (at 35.7251 65.0748) (layer F.SilkS)
     (effects (font (size 1 1) (thickness 0.2)))
   )
